Commit message: week2 WIP

File: src/week2/description/urdf/simple_robot.urdf.xacro (robot description, xacro)
@@ -1,8 +1,7 @@
 <robot name="simple_robot" xmlns:xacro="http://www.ros.org/wiki/xacro">
-  <link name="world">
-  </link>
+  <link name="world"/>
   <link name="base_link"> <!-- Each link should have a name to distinguish and refer to them -->
     <visual>
-      <origin xyz="0 0 0.3" rpy="0 0 0"/>
+      <origin xyz="0 0 0.1" rpy="0 0 0"/>
       <geometry>
         <box size="0.2 0.2 0.2"/> <!-- This specifies the shape of the link -->
@@ -25,11 +24,11 @@
   </link>
   <joint name="fixed" type="fixed">
-    <origin xyz="2.5 -1 0" rpy="0 0 0"/>
+    <origin xyz="2.5 -1 0" rpy="0 0 0"/> <!-- Rotate and offset the link (not its geometry) -->
     <parent link="world"/>
     <child link="base_link"/>
   </joint>
   <joint name="base_to_link_1" type="continuous">
-    <origin xyz="0 0 0.2" rpy="${pi/2} 0 0"/>
-    <axis xyz="0 1 0"/>
+    <origin xyz="0 0 0.2" rpy="${pi/2} 0 0"/> <!-- Rotate and offset the link (not its geometry) -->
+    <axis xyz="0 1 0"/> <!-- This is the axis of rotation, by default rotation is on the x axis-->
     <parent link="base_link"/>
     <child link="link_1"/>
