Commit message: fixed frame 6dof

File: src/week2/description/urdf/6dof.urdf.xacro (robot description, xacro)
@@ -1,4 +1,4 @@
 <robot name="fanuc_cr7ia"  xmlns:xacro="http://wiki.ros.org/xacro">
-    <!-- links: main serial chain -->
+    <link name="world"/>
     <link name="base_link">
       <visual>
@@ -11,10 +11,4 @@
         </material>
       </visual>
-      <!-- <collision>
-        <origin xyz="0 0 0" rpy="0 0 0"/>
-        <geometry>
-          <mesh filename="package://week2/description/meshes/collision/base_link.stl"/>
-        </geometry>
-      </collision> -->
     </link>
     <link name="link_1">
@@ -28,10 +22,4 @@
         </material>
       </visual>
-      <!-- <collision>
-        <origin xyz="0 0 0" rpy="0 0 0"/>
-        <geometry>
-          <mesh filename="package://week2/description/meshes/collision/link_1.stl"/>
-        </geometry>
-      </collision> -->
     </link>
     <link name="link_2">
@@ -45,10 +33,4 @@
         </material>
       </visual>
-      <!-- <collision>
-        <origin xyz="0 0 0" rpy="0 0 0"/>
-        <geometry>
-          <mesh filename="package://week2/description/meshes/collision/link_2.stl"/>
-        </geometry>
-      </collision> -->
     </link>
     <link name="link_3">
@@ -62,10 +44,4 @@
         </material>
       </visual>
-      <!-- <collision>
-        <origin xyz="0 0 0" rpy="0 0 0"/>
-        <geometry>
-          <mesh filename="package://week2/description/meshes/collision/link_3.stl"/>
-        </geometry>
-      </collision> -->
     </link>
     <link name="link_4">
@@ -79,10 +55,4 @@
         </material>
       </visual>
-      <!-- <collision>
-        <origin xyz="0 0 0" rpy="0 0 0"/>
-        <geometry>
-          <mesh filename="package://week2/description/meshes/collision/link_4.stl"/>
-        </geometry>
-      </collision> -->
     </link>
     <link name="link_5">
@@ -96,10 +66,4 @@
         </material>
       </visual>
-      <!-- <collision>
-        <origin xyz="0 0 0" rpy="0 0 0"/>
-        <geometry>
-          <mesh filename="package://week2/description/meshes/collision/link_5.stl"/>
-        </geometry>
-      </collision> -->
     </link>
     <link name="link_6">
@@ -113,10 +77,4 @@
         </material>
       </visual>
-      <!-- <collision>
-        <origin xyz="0 0 0" rpy="0 0 0"/>
-        <geometry>
-          <mesh filename="package://week2/description/meshes/collision/link_6.stl"/>
-        </geometry>
-      </collision> -->
     </link>
     <!-- joints: main serial chain -->
@@ -163,24 +121,8 @@
       <limit effort="0" lower="-6.2832" upper="6.2832" velocity="17.4532" />
     </joint>
-    <!-- ROS-Industrial 'base' frame: base_link to Fanuc World Coordinates transform -->
-    <link name="base" />
-    <joint name="base_link-base" type="fixed">
-      <origin xyz="0 0 0.457" rpy="0 0 0"/>
-      <parent link="base_link"/>
-      <child link="base"/>
-    </joint>
-    <!-- ROS-Industrial 'flange' frame: attachment point for EEF models -->
-    <link name="flange" />
-    <joint name="joint_6-flange" type="fixed">
-      <origin xyz="0 0 0" rpy="0 0 0" />
-      <parent link="link_6" />
-      <child link="flange" />
-    </joint>
-    <!-- ROS-Industrial 'tool0' frame: all-zeros tool frame -->
-    <link name="tool0" />
-    <joint name="link_6-tool0" type="fixed">
-      <origin xyz="0 0 0" rpy="${pi} ${-pi/2.0} 0" />
-      <parent link="flange" />
-      <child link="tool0" />
+    <joint name="fixed" type="fixed">
+      <origin xyz="0 0 0" rpy="0 0 0"/>
+      <parent link="world"/>
+      <child link="base_link"/>
     </joint>
 </robot>

Commit message: removing things not needed for workshop

File: src/week2/description/urdf/6dof.urdf.xacro (robot description, xacro)
@@ -8,5 +8,5 @@
         </geometry>
         <material name="base_material">
-          <color rgba="0.34 0.35 0.36 1.0"/> <!-- This specifies the color of the link -->
+          <color rgba="0.34 0.35 0.36 1.0"/>
         </material>
       </visual>
@@ -19,5 +19,5 @@
         </geometry>
         <material name="link_1_material">
-          <color rgba="${  0/255} ${155/255} ${ 70/255} 1.0"/> <!-- This specifies the color of the link -->
+          <color rgba="${  0/255} ${155/255} ${ 70/255} 1.0"/>
         </material>
       </visual>
@@ -30,5 +30,5 @@
         </geometry>
         <material name="link_2_material">
-          <color rgba=" ${  0/255} ${155/255} ${ 70/255} 1.0"/> <!-- This specifies the color of the link -->
+          <color rgba=" ${  0/255} ${155/255} ${ 70/255} 1.0"/>
         </material>
       </visual>
@@ -41,5 +41,5 @@
         </geometry>
         <material name="link_3_material">
-          <color rgba="${  0/255} ${155/255} ${ 70/255} 1.0"/> <!-- This specifies the color of the link -->
+          <color rgba="${  0/255} ${155/255} ${ 70/255} 1.0"/>
         </material>
       </visual>
@@ -52,5 +52,5 @@
         </geometry>
         <material name="link_4_material">
-          <color rgba="${  0/255} ${155/255} ${ 70/255} 1.0"/> <!-- This specifies the color of the link -->
+          <color rgba="${  0/255} ${155/255} ${ 70/255} 1.0"/>
         </material>
       </visual>
@@ -63,5 +63,5 @@
         </geometry>
         <material name="link_5_material">
-          <color rgba="${  0/255} ${155/255} ${ 70/255} 1.0"/> <!-- This specifies the color of the link -->
+          <color rgba="${  0/255} ${155/255} ${ 70/255} 1.0"/>
         </material>
       </visual>
@@ -74,5 +74,5 @@
         </geometry>
         <material name="link_6_material">
-          <color rgba="0.34 0.35 0.36 1.0"/> <!-- This specifies the color of the link -->
+          <color rgba="0.34 0.35 0.36 1.0"/>
         </material>
       </visual>
@@ -80,43 +80,43 @@
     <!-- joints: main serial chain -->
     <joint name="joint_1" type="revolute">
-      <origin xyz="0 0 0.457" rpy="0 0 0" />
+      <origin xyz="0 0 1" rpy="0 0 0"/>
       <parent link="base_link" />
       <child link="link_1" />
-      <axis xyz="0 0 1" />
+      <axis xyz="1 0 0" />
       <limit effort="0" lower="-2.9671" upper="2.9671" velocity="7.8539" />
     </joint>
     <joint name="joint_2" type="revolute">
-      <origin xyz="0.05 0 0" rpy="0 0 0" />
+      <origin xyz="0 0 1" rpy="0 0 0"/>
       <parent link="link_1" />
       <child link="link_2" />
-      <axis xyz="0 1 0" />
+      <axis xyz="1 0 0" />
       <limit effort="0" lower="-1.1519" upper="1.7453" velocity="6.6322" />
     </joint>
     <joint name="joint_3" type="revolute">
-      <origin xyz="0 0 0.330" rpy="0 0 0" />
+      <origin xyz="0 0 1" rpy="0 0 0"/>
       <parent link="link_2" />
       <child link="link_3" />
-      <axis xyz="0 -1 0" />
+      <axis xyz="1 0 0" />
       <limit effort="0" lower="-2.2621" upper="4.2586" velocity="9.0757" />
     </joint>
     <joint name="joint_4" type="revolute">
-      <origin xyz="0 0 0.035" rpy="0 0 0"/>
+      <origin xyz="0 0 1" rpy="0 0 0"/>
       <parent link="link_3"/>
       <child link="link_4"/>
-      <axis xyz="-1 0 0"/>
+      <axis xyz="1 0 0" />
       <limit effort="0" lower="-3.3161" upper="3.3161" velocity="9.5993" />
     </joint>
     <joint name="joint_5" type="revolute">
-      <origin xyz="0.335 0 0" rpy="0 0 0"/>
+      <origin xyz="0 0 1" rpy="0 0 0"/>
       <parent link="link_4"/>
       <child link="link_5"/>
-      <axis xyz="0 -1 0"/>
+      <axis xyz="1 0 0" />
       <limit effort="0" lower="-2.0944" upper="2.0944" velocity="9.5120" />
     </joint>
     <joint name="joint_6" type="revolute">
-      <origin xyz="0.080 0 0" rpy="0 0 0"/>
+      <origin xyz="0 0 1" rpy="0 0 0"/>
       <parent link="link_5"/>
       <child link="link_6"/>
-      <axis xyz="-1 0 0"/>
+      <axis xyz="1 0 0" />
       <limit effort="0" lower="-6.2832" upper="6.2832" velocity="17.4532" />
     </joint>

Commit message: WIP week4

File: src/week2/description/urdf/6dof.urdf.xacro (robot description, xacro)
@@ -1,128 +1,142 @@
-<robot name="fanuc_cr7ia"  xmlns:xacro="http://wiki.ros.org/xacro">
-    <link name="world"/>
-    <link name="base_link">
-      <visual>
-        <origin xyz="0 0 0" rpy="0 0 0"/>
-        <geometry>
-          <mesh filename="package://week2/description/meshes/visual/base_link.stl"/>
-        </geometry>
-        <material name="base_material">
-          <color rgba="0.34 0.35 0.36 1.0"/>
-        </material>
-      </visual>
-    </link>
-    <link name="link_1">
-      <visual>
-        <origin xyz="0 0 0" rpy="0 0 0"/>
-        <geometry>
-          <mesh filename="package://week2/description/meshes/visual/link_1.stl"/>
-        </geometry>
-        <material name="link_1_material">
-          <color rgba="${  0/255} ${155/255} ${ 70/255} 1.0"/>
-        </material>
-      </visual>
-    </link>
-    <link name="link_2">
-      <visual>
-        <origin xyz="0 0 0" rpy="0 0 0"/>
-        <geometry>
-          <mesh filename="package://week2/description/meshes/visual/link_2.stl"/>
-        </geometry>
-        <material name="link_2_material">
-          <color rgba=" ${  0/255} ${155/255} ${ 70/255} 1.0"/>
-        </material>
-      </visual>
-    </link>
-    <link name="link_3">
-      <visual>
-        <origin xyz="0 0 0" rpy="0 0 0"/>
-        <geometry>
-          <mesh filename="package://week2/description/meshes/visual/link_3.stl"/>
-        </geometry>
-        <material name="link_3_material">
-          <color rgba="${  0/255} ${155/255} ${ 70/255} 1.0"/>
-        </material>
-      </visual>
-    </link>
-    <link name="link_4">
-      <visual>
-        <origin xyz="0 0 0" rpy="0 0 0"/>
-        <geometry>
-          <mesh filename="package://week2/description/meshes/visual/link_4.stl"/>
-        </geometry>
-        <material name="link_4_material">
-          <color rgba="${  0/255} ${155/255} ${ 70/255} 1.0"/>
-        </material>
-      </visual>
-    </link>
-    <link name="link_5">
-      <visual>
-        <origin xyz="0 0 0" rpy="0 0 0"/>
-        <geometry>
-          <mesh filename="package://week2/description/meshes/visual/link_5.stl"/>
-        </geometry>
-        <material name="link_5_material">
-          <color rgba="${  0/255} ${155/255} ${ 70/255} 1.0"/>
-        </material>
-      </visual>
-    </link>
-    <link name="link_6">
-      <visual>
-        <origin xyz="0 0 0" rpy="0 0 0"/>
-        <geometry>
-          <mesh filename="package://week2/description/meshes/visual/link_6.stl"/>
-        </geometry>
-        <material name="link_6_material">
-          <color rgba="0.34 0.35 0.36 1.0"/>
-        </material>
-      </visual>
-    </link>
-    <!-- joints: main serial chain -->
-    <joint name="joint_1" type="revolute">
-      <origin xyz="0 0 1" rpy="0 0 0"/>
-      <parent link="base_link" />
-      <child link="link_1" />
-      <axis xyz="1 0 0" />
-      <limit effort="0" lower="-2.9671" upper="2.9671" velocity="7.8539" />
-    </joint>
-    <joint name="joint_2" type="revolute">
-      <origin xyz="0 0 1" rpy="0 0 0"/>
-      <parent link="link_1" />
-      <child link="link_2" />
-      <axis xyz="1 0 0" />
-      <limit effort="0" lower="-1.1519" upper="1.7453" velocity="6.6322" />
-    </joint>
-    <joint name="joint_3" type="revolute">
-      <origin xyz="0 0 1" rpy="0 0 0"/>
-      <parent link="link_2" />
-      <child link="link_3" />
-      <axis xyz="1 0 0" />
-      <limit effort="0" lower="-2.2621" upper="4.2586" velocity="9.0757" />
-    </joint>
-    <joint name="joint_4" type="revolute">
-      <origin xyz="0 0 1" rpy="0 0 0"/>
-      <parent link="link_3"/>
-      <child link="link_4"/>
-      <axis xyz="1 0 0" />
-      <limit effort="0" lower="-3.3161" upper="3.3161" velocity="9.5993" />
-    </joint>
-    <joint name="joint_5" type="revolute">
-      <origin xyz="0 0 1" rpy="0 0 0"/>
-      <parent link="link_4"/>
-      <child link="link_5"/>
-      <axis xyz="1 0 0" />
-      <limit effort="0" lower="-2.0944" upper="2.0944" velocity="9.5120" />
-    </joint>
-    <joint name="joint_6" type="revolute">
-      <origin xyz="0 0 1" rpy="0 0 0"/>
-      <parent link="link_5"/>
-      <child link="link_6"/>
-      <axis xyz="1 0 0" />
-      <limit effort="0" lower="-6.2832" upper="6.2832" velocity="17.4532" />
-    </joint>
-    <joint name="fixed" type="fixed">
+<robot name="fanuc_cr7ia"
+  xmlns:xacro="http://wiki.ros.org/xacro">
+  <link name="world"/>
+  <link name="base_link">
+    <visual>
       <origin xyz="0 0 0" rpy="0 0 0"/>
-      <parent link="world"/>
-      <child link="base_link"/>
-    </joint>
+      <geometry>
+        <mesh filename="package://week2/description/meshes/visual/base_link.stl"/>
+      </geometry>
+      <material name="base_material">
+        <color rgba="0.34 0.35 0.36 1.0"/>
+        <!-- This specifies the color of the link -->
+      </material>
+    </visual>
+  </link>
+  <link name="link_1">
+    <visual>
+      <origin xyz="0 0 0" rpy="0 0 0"/>
+      <geometry>
+        <mesh filename="package://week2/description/meshes/visual/link_1.stl"/>
+      </geometry>
+      <material name="link_1_material">
+        <color rgba="${  0/255} ${155/255} ${ 70/255} 1.0"/>
+        <!-- This specifies the color of the link -->
+      </material>
+    </visual>
+  </link>
+  <link name="link_2">
+    <visual>
+      <origin xyz="0 0 0" rpy="0 0 0"/>
+      <geometry>
+        <mesh filename="package://week2/description/meshes/visual/link_2.stl"/>
+      </geometry>
+      <material name="link_2_material">
+        <color rgba=" ${  0/255} ${155/255} ${ 70/255} 1.0"/>
+        <!-- This specifies the color of the link -->
+      </material>
+    </visual>
+  </link>
+  <link name="link_3">
+    <visual>
+      <origin xyz="0 0 0" rpy="0 0 0"/>
+      <geometry>
+        <mesh filename="package://week2/description/meshes/visual/link_3.stl"/>
+      </geometry>
+      <material name="link_3_material">
+        <color rgba="${  0/255} ${155/255} ${ 70/255} 1.0"/>
+        <!-- This specifies the color of the link -->
+      </material>
+    </visual>
+  </link>
+  <link name="link_4">
+    <visual>
+      <origin xyz="0 0 0" rpy="0 0 0"/>
+      <geometry>
+        <mesh filename="package://week2/description/meshes/visual/link_4.stl"/>
+      </geometry>
+      <material name="link_4_material">
+        <color rgba="${  0/255} ${155/255} ${ 70/255} 1.0"/>
+        <!-- This specifies the color of the link -->
+      </material>
+    </visual>
+  </link>
+  <link name="link_5">
+    <visual>
+      <origin xyz="0 0 0" rpy="0 0 0"/>
+      <geometry>
+        <mesh filename="package://week2/description/meshes/visual/link_5.stl"/>
+      </geometry>
+      <material name="link_5_material">
+        <color rgba="${  0/255} ${155/255} ${ 70/255} 1.0"/>
+        <!-- This specifies the color of the link -->
+      </material>
+    </visual>
+  </link>
+  <link name="link_6">
+    <visual>
+      <origin xyz="0 0 0" rpy="0 0 0"/>
+      <geometry>
+        <mesh filename="package://week2/description/meshes/visual/link_6.stl"/>
+      </geometry>
+      <material name="link_6_material">
+        <color rgba="0.34 0.35 0.36 1.0"/>
+        <!-- This specifies the color of the link -->
+      </material>
+    </visual>
+  </link>
+  <link name="tool_link"/>
+  <!-- joints: main serial chain -->
+  <joint name="joint_1" type="revolute">
+    <origin xyz="0 0 0.457" rpy="0 0 0" />
+    <parent link="base_link" />
+    <child link="link_1" />
+    <axis xyz="0 0 1" />
+    <limit effort="0" lower="-2.9671" upper="2.9671" velocity="7.8539" />
+  </joint>
+  <joint name="joint_2" type="revolute">
+    <origin xyz="0.05 0 0" rpy="0 0 0" />
+    <parent link="link_1" />
+    <child link="link_2" />
+    <axis xyz="0 1 0" />
+    <limit effort="0" lower="-1.1519" upper="1.7453" velocity="6.6322" />
+  </joint>
+  <joint name="joint_3" type="revolute">
+    <origin xyz="0 0 0.330" rpy="0 0 0" />
+    <parent link="link_2" />
+    <child link="link_3" />
+    <axis xyz="0 -1 0" />
+    <limit effort="0" lower="-2.2621" upper="4.2586" velocity="9.0757" />
+  </joint>
+  <joint name="joint_4" type="revolute">
+    <origin xyz="0 0 0.035" rpy="0 0 0"/>
+    <parent link="link_3"/>
+    <child link="link_4"/>
+    <axis xyz="-1 0 0"/>
+    <limit effort="0" lower="-3.3161" upper="3.3161" velocity="9.5993" />
+  </joint>
+  <joint name="joint_5" type="revolute">
+    <origin xyz="0.335 0 0" rpy="0 0 0"/>
+    <parent link="link_4"/>
+    <child link="link_5"/>
+    <axis xyz="0 -1 0"/>
+    <limit effort="0" lower="-2.0944" upper="2.0944" velocity="9.5120" />
+  </joint>
+  <joint name="joint_6" type="revolute">
+    <origin xyz="0.080 0 0" rpy="0 0 0"/>
+    <parent link="link_5"/>
+    <child link="link_6"/>
+    <axis xyz="-1 0 0"/>
+    <limit effort="0" lower="-6.2832" upper="6.2832" velocity="17.4532" />
+  </joint>
+  <joint name="fixed" type="fixed">
+    <origin xyz="0 0 0" rpy="0 0 0"/>
+    <parent link="world"/>
+    <child link="base_link"/>
+  </joint>
+  <joint name="fixed_tool" type="fixed">
+    <origin xyz="0.08 0 0" rpy="0 0 0"/>
+    <parent link="link_6"/>
+    <child link="tool_link"/>
+  </joint>
 </robot>

Commit message: WIP not working

File: src/week2/description/urdf/6dof.urdf.xacro (robot description, xacro)
@@ -136,5 +136,5 @@
   </joint>
   <joint name="fixed_tool" type="fixed">
-    <origin xyz="0.08 0 0" rpy="0 0 0"/>
+    <origin xyz="0 0 0" rpy="0 0 0"/>
     <parent link="link_6"/>
     <child link="tool_link"/>
