Commit message: fixed launch file for gazebo and controllers

File: src/mecharm_description/urdf/firefighter.urdf.xacro (robot description, xacro)
@@ -1,9 +1,24 @@
 <?xml version="1.0"?>
 <robot xmlns:xacro="http://www.ros.org/wiki/xacro" name="firefighter">
-    <xacro:arg name="initial_positions_file" default="$(find mecharm_moveit_config)/config/initial_positions.yaml" />
+    <xacro:arg name="robot_name" default="firefighter"/>
+    <xacro:arg name="use_gazebo" default="true"/>
+    <!-- <xacro:arg name="initial_positions_file" default="$(find mecharm_moveit_config)/config/initial_positions.yaml" /> -->
     <!-- Import firefighter urdf file -->
-    <xacro:include filename="$(find mycobot_description)/urdf/mecharm_270_m5/mecharm_270_m5.urdf" />
+    <xacro:include filename="$(find mecharm_description)/urdf/mecharm_270_m5.urdf" />
+    <xacro:mecharm>
+      <origin xyz="0 0 0" rpy="0 0 0"/>
+    </xacro:mecharm>
     <!-- Import control_xacro -->
     <xacro:include filename="$(find mecharm_moveit_config)/config/firefighter.ros2_control.xacro" />
-    <xacro:firefighter_ros2_control name="FakeSystem" initial_positions_file="$(arg initial_positions_file)"/>
+    <!-- <xacro:firefighter_ros2_control
+            name="FakeSystem"
+            initial_positions_file="$(arg initial_positions_file)"
+            use_gazebo="true"/> -->
+    <xacro:firefighter_ros2_control
+            name="FakeSystem"
+            use_gazebo="$(arg use_gazebo)"/>
+    <xacro:include filename="$(find mecharm_moveit_config)/config/gazebo_sim_ros2_control.urdf.xacro" />
+    <xacro:load_gazebo_sim_ros2_control_plugin
+      robot_name="$(arg robot_name)"
+      use_gazebo="$(arg use_gazebo)"/>
 </robot>

File: src/mecharm_moveit_config/config/firefighter.ros2_control.xacro (robot description, xacro)
@@ -1,52 +1,69 @@
 <?xml version="1.0"?>
 <robot xmlns:xacro="http://www.ros.org/wiki/xacro">
-    <xacro:macro name="firefighter_ros2_control" params="name initial_positions_file">
-        <xacro:property name="initial_positions" value="${load_yaml(initial_positions_file)['initial_positions']}"/>
+    <xacro:macro name="firefighter_ros2_control" params="name use_gazebo">
+        <!-- <xacro:property name="initial_positions" value="${load_yaml(initial_positions_file)['initial_positions']}"/> -->
         <ros2_control name="${name}" type="system">
             <hardware>
                 <!-- By default, set up controllers for simulation. This won't work on real hardware -->
-                <plugin>mock_components/GenericSystem</plugin>
+                <xacro:if value="${use_gazebo}">
+                    <plugin>ign_ros2_control/IgnitionSystem</plugin>
+                </xacro:if>
+                <xacro:unless value="${use_gazebo}">
+                  <plugin>mock_components/GenericSystem</plugin>
+                </xacro:unless>
             </hardware>
             <joint name="joint1_to_base">
                 <command_interface name="position"/>
-                <state_interface name="position">
+                <command_interface name="velocity"/>
+                <!-- <state_interface name="position">
                   <param name="initial_value">${initial_positions['joint1_to_base']}</param>
-                </state_interface>
+                </state_interface> -->
                 <state_interface name="velocity"/>
+                <state_interface name="position"/>
             </joint>
             <joint name="joint2_to_joint1">
                 <command_interface name="position"/>
-                <state_interface name="position">
+                <command_interface name="velocity"/>
+                <!-- <state_interface name="position">
                   <param name="initial_value">${initial_positions['joint2_to_joint1']}</param>
-                </state_interface>
+                </state_interface> -->
                 <state_interface name="velocity"/>
+                <state_interface name="position"/>
             </joint>
             <joint name="joint3_to_joint2">
                 <command_interface name="position"/>
-                <state_interface name="position">
+                <command_interface name="velocity"/>
+                <!-- <state_interface name="position">
                   <param name="initial_value">${initial_positions['joint3_to_joint2']}</param>
-                </state_interface>
+                </state_interface> -->
                 <state_interface name="velocity"/>
+                <state_interface name="position"/>
             </joint>
             <joint name="joint4_to_joint3">
                 <command_interface name="position"/>
-                <state_interface name="position">
+                <command_interface name="velocity"/>
+                <!-- <state_interface name="position">
                   <param name="initial_value">${initial_positions['joint4_to_joint3']}</param>
-                </state_interface>
+                </state_interface> -->
                 <state_interface name="velocity"/>
+                <state_interface name="position"/>
             </joint>
             <joint name="joint5_to_joint4">
                 <command_interface name="position"/>
-                <state_interface name="position">
+                <command_interface name="velocity"/>
+                <!-- <state_interface name="position">
                   <param name="initial_value">${initial_positions['joint5_to_joint4']}</param>
-                </state_interface>
+                </state_interface> -->
                 <state_interface name="velocity"/>
+                <state_interface name="position"/>
             </joint>
             <joint name="joint6_to_joint5">
                 <command_interface name="position"/>
-                <state_interface name="position">
+                <command_interface name="velocity"/>
+                <!-- <state_interface name="position">
                   <param name="initial_value">${initial_positions['joint6_to_joint5']}</param>
-                </state_interface>
+                </state_interface> -->
                 <state_interface name="velocity"/>
+                <state_interface name="position"/>
             </joint>
         </ros2_control>
